File: hardware/ACme++/rev_a/ACme++.sch (EAGLE design)
At the start: 52 parts, among them J3 MA02-1, SW1 SWITCH_SPDP, T1 NCHAN_MOSFET, T2 NCHAN_MOSFET, T3 NCHAN_MOSFET, U1 ADE7753, U2 LTC3588_, U3 FM25LB, X1 ECS-35-17-5PX-TR

Commit message: working on relay
Parts:
- removed C13: 0.1uF, rcl:C-EUC0603
- removed R24, R25, R26: 4.7k, rcl:R-US_R0603
- removed TP11, TP12, TP7: WHITE, con-lstb:MA01-1
- removed TP13: GREEN, con-lstb:MA01-1
- removed U3: FM25LB, coilcube:FM25LB
- added D1: DIODE_MMBD914, powercube:DIODE_MMBD914
- added K1: S216S01F, powercube:S216S01F
- added R10: 100k, SparkFun:RESISTOR0603-RES
- added R9: (no value), SparkFun-Resistors:RESISTOR0805-RES
- added U$1: FDV301N, powercube:FDV301N
Connections:
- removed net FRAM_CS: R24.1, TP13.1, U3.!CS
- removed net FRAM_HOLD: R25.1, U3.!HOLD
- removed net FRAM_WP: R26.1, U3.!WP
- removed net MISO0: TP11.1, U3.SO
- removed net MOSI0: TP7.1, U3.SI
- removed net SCK0: TP12.1, U3.SCK
- new net N$13: D1.1, K1.3, R9.1
- new net N$4: D1.2, K1.4, U$1.D
- new net RELAY_CTRL: R10.2, U$1.G
- net +3V3: no longer C13.1, R24.2, R25.2, R26.2, U3.VDD
- net 3V3: now also R10.1
- net 5V: now also R9.2
- net GND: now also U$1.S; no longer C13.2, U3.VSS

Commit message: working on ac connections
Parts:
- added C13, C22, C23: 33nF, SparkFun-Passives:CAP0805
- added J1: AC-PLUG, powercube:AC-PLUG
- added J2, J4, J5: WIRE_HOLE-14AWG, powercube:WIRE_HOLE-14AWG
- added L2, L3: EMI_SUPRESSION_FERRITE_BEAD, powercube:EMI_SUPRESSION_FERRITE_BEAD
- added L4: 35F0121-0SR-10, powercube:35F0121-0SR-10
- added R11: .001, SparkFun-Resistors:RESISTOR2512
- added R12, R13: 1k, SparkFun-Resistors:RESISTOR0805-RES
- added R14: 499k, SparkFun-Resistors:RESISTOR0805-RES
- added R15: 1k, SparkFun-Resistors:RESISTOR0603-RES
Connections:
- new net EARTH_GND: J1.GND, J5.P$1
- new net LOAD_NEUTRAL: J4.P$1, L3.P$1, R11.2
- new net LOAD_PHASE: J2.P$1, K1.2
- new net N$14: L2.P$2, R12.1
- new net N$16: L3.P$2, R13.1
- new net N$17: L4.P$2, R14.1
- new net WALL_NEUTRAL: J1.NEUTRAL, L2.P$1, R11.1
- new net WALL_PHASE: J1.PHASE, K1.1, L4.P$1
- net GND: now also C13.2, C22.2, C23.2, R15.1
- net V1N: now also C13.1, R12.2
- net V1P: now also C22.1, R13.2
- net V2P: now also C23.1, R14.2, R15.2
Other:
- note added: "Sense Resistor"
- moved on the sheet: K1, R10, R9, U$1

Commit message: power supplies fleshed out
Parts:
- removed C12: 2.2uF, coilcube:CAP_POLEA1MM5
- removed C16: 47uF, SparkFun-Passives:CAP_POL1206
- removed C18, C19, C20: 100uF 25V, coilcube:2917_CAP_POL
- removed C21: 0.1uF, rcl:C-EUC0603
- removed J3: MA02-1, con-lstb:MA02-1
- removed L1: 10uH, SparkFun-Passives:INDUCTOR1210
- removed R3: 10k, SparkFun:RESISTOR0603-RES
- removed S2: SWITCH-OFF-MOM, p498:SWITCH-OFF-MOM
- removed SW1: SWITCH_SPDP, coilcube:SWITCH_SPDP
- removed T1, T2, T3: NCHAN_MOSFET, Power_Metering:NCHAN_MOSFET
- removed TP1: ORANGE, con-lstb:MA01-1
- removed TP16: RED, con-lstb:MA01-1
- removed TP17: BLACK, con-lstb:MA01-1
- removed TP6: BLUE, con-lstb:MA01-1
- added D2: SMAJ_TVS, powercube:SMAJ_TVS
- added D3: CD2320-BB11000, powercube:CD2320-BB11000
- added Q1: STGD5NB120SZT4, powercube:STGD5NB120SZT4
- added R17: 113k, SparkFun-Resistors:RESISTOR0603-RES
- added R18: 12.4k, SparkFun-Resistors:RESISTOR0603-RES
- added S1: EVQP2, epic:EVQP2
- added U3: TDA3664AT, powercube:TDA3664AT
- C10: device rcl:C-EUC0603 -> SparkFun-Passives:CAP0603-CAP
- C11: value 10uF -> 47uF; device rcl:C-EUC1206 -> SparkFun-Passives:CAP1206; DIGIKEY 399-8152-1-ND -> 399-5508-1-ND
- C5: value 100uF 25V -> 1uF; device coilcube:2917_CAP_POL -> SparkFun-Passives:CAP0603-CAP; DIGIKEY 399-5175-1-ND -> 445-5956-1-ND
- C6: value 100uF 25V -> 1uF; device coilcube:2917_CAP_POL -> SparkFun-Passives:CAP1206; DIGIKEY 399-5175-1-ND -> 445-1381-1-ND
- C7: value 1uF -> 470uF; device rcl:C-EUC0603 -> powercube:CAP_EEE-FP1E471AP; DIGIKEY 445-1321-1-ND -> (none)
- C8: value 4.7uF -> 0.1uF; device rcl:C-EUC0603 -> SparkFun-Passives:CAP0603-CAP; DIGIKEY 445-5178-1-ND -> (none)
- R1: value 0 -> 200k; device rcl:R-US_R0603 -> SparkFun-Resistors:RESISTOR1206; DIGIKEY P0.0GCT-ND -> P200KALCT-ND
- R2: value NP -> 200k; device rcl:R-US_R0603 -> SparkFun-Resistors:RESISTOR1206; DIGIKEY (none) -> P200KALCT-ND
- R4: value 4.7M -> 510k; device rcl:R-US_R0805 -> SparkFun-Resistors:RESISTOR1206; DIGIKEY P4.7MACT-ND -> P510KALCT-ND
- R5: value NP -> 510k; device rcl:R-US_R0603 -> SparkFun-Resistors:RESISTOR1206; DIGIKEY (none) -> P510KALCT-ND
- R7: value 0 -> 10k; device rcl:R-US_R0603 -> SparkFun:RESISTOR0603-RES; DIGIKEY P0.0GCT-ND -> P10KGCT-ND
- U2: value LTC3588_ -> SR086SG-G; device SparkFun-PowerIC:LTC3588_ -> powercube:SR086SG-G; DIGIKEY LTC3588EMSE-1#PBF-ND -> (none)
Connections:
- removed net +3V3: C11.1, C16.+, C21.1, L1.2, T1.G, T2.D, T3.G, TP16.1, U2.VOUT
- removed net D0: R5.1, R7.1, U2.D0
- removed net D1: R1.1, R2.1, U2.D1
- removed net FTDIVDD: R3.2
- removed net N$2: S2.P1, S2.P3
- removed net N$20: L1.1, U2.SW
- removed net PGOOD: U2.PGOOD
- removed net PZ1: J3.2, T1.D, U2.PZ1
- removed net PZ2: SW1.P1, U2.PZ2
- removed net RST: R3.1, S2.P2, S2.P4
- removed net TIME_CTL: T2.G
- removed net VCAP: C10.1, C18.+, C19.+, C20.+, C5.+, C6.+, C7.1, TP1.1, U2.VIN
- removed net VIN2: C8.1, R1.2, R5.2, U2.VIN2
- removed net VTIMER: C12.+, R4.2, T2.S, TP6.1
- new net 5V0: C11.1, U3.VOUT
- new net N$18: R1.1, R2.2
- new net N$19: R5.1, U2.VIN
- new net N$21: R4.1, R5.2
- new net N$24: C10.2, U2.VGD
- new net N$26: R17.1, R18.2, U2.FB
- new net USER_RELAY_CTRL: R7.2, S1.P$2, S1.P$4
- new net VDC: C10.1, C5.1, C6.1, C7.+, Q1.E, R17.2, U2.VOUT, U3.VIN
- net 3V3: now also C8.1, S1.P$1, S1.P$3, U2.VREG
- net GND: now also C5.2, C6.2, C7.-, D3.NEG, R18.1, R2.1, R7.1, U2.!EN, U3.GND; no longer C10.2, C12.-, C16.-, C18.-, C19.-, C20.-, C21.2, C5.-, C6.-, R2.2, R4.1, R7.2, SW1.P2, T1.S, T3.S, TP17.1
- net N$1: now also D3.POS, Q1.C, R1.2, R4.2; no longer J3.1, SW1.PC, T3.D
- net N$22: now also Q1.G, U2.GATE; no longer C7.2, U2.CAP
- net WALL_NEUTRAL: now also D2.P$2, D3.AC2
- net WALL_PHASE: now also D2.P$1, D3.AC1
Other:
- note added: "5V Regulator"
- note added: "AC-DC Converter"
- note added: "Nominally 12.6 V"
- note removed: "Output Voltage Selection"

Commit message: progress
cleaned up schematic a bit

initial arragnment on pcb
Parts:
- renumbered U$1 to Q2
Connections:
- removed net 5V: C1.1, C2.1, R6.2, R8.1, R9.2, U1.DVDD
- removed net N$10: JP1.8
- removed net N$6: JP1.4
- removed net N$7: JP1.5
- removed net N$8: JP1.6
- removed net N$9: JP1.7
- removed net V2N: U1.V2N
- net !ADE_CS: now also JP1.4
- net !ADE_IRQ: now also JP1.5
- net 5V0: now also C1.1, C2.1, R6.2, R8.1, R9.2, U1.DVDD
- net ADE_CF: now also JP1.7
- net ADE_ZX: now also JP1.6
- net USER_RELAY_CTRL: now also JP1.8
- net V1N: now also U1.V2N
Other:
- moved on the sheet: R9

Commit message: working on routing
power supply laid out

working on ace

lots of room...put cc2538 on this board? hard to argue not to...
Connections:
- net N$1 renamed DC_RECTIFIED
- net N$19 renamed SR086_VIN
- net N$22 renamed SR086_GATE
Changed lines of the file:
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@@
 </segment>
 </net>
-<net name="N$1" class="0">
+<net name="DC_RECTIFIED" class="0">
 <segment>
 <pinref part="D3" gate="G$1" pin="POS"/>
@@
 </segment>
 </net>
-<net name="N$19" class="0">
+<net name="SR086_VIN" class="0">
 <segment>
 <pinref part="U2" gate="G$1" pin="VIN"/>
@@
 </segment>
 </net>
-<net name="N$22" class="0">
+<net name="SR086_GATE" class="0">
 <segment>
 <pinref part="Q1" gate="G$1" pin="G"/>

Commit message: routing the cc2538
Parts:
- removed JP1: (no value), pinhead:PINHD-1X12
- added A1: FRACTUS-2.4GHZ-FR05-S1-N-0-001, chips:FRACTUS-2.4GHZ-FR05-S1-N-0-001
- added B1: 2450BM15A0002, chips:2450BM15A0002
- added C12, C16: 12pF, passives:CAPACITOR
- added C18, C29, C30: 1uF, passives:CAPACITOR
- added C19, C20, C21, C24, C25, C27, C28, C31: 0.1uF, passives:CAPACITOR
- added C26: 220pF, passives:CAPACITOR
- added C32: 1nF, passives:CAPACITOR
- added C33, C34: 22pF, passives:CAPACITOR
- added J3: TC2030-CTX-NL, connector:TC2030-CTX-NL
- added R16, R19, R3: 4.7k, passives:RESISTOR
- added R20, R22: 2.2k, passives:RESISTOR
- added R21: 56k, passives:RESISTOR
- added U4: FM25LBTDFN-8, chips:FM25LBTDFN-8
- added U5: CC2538, chips:CC2538
- added U6: DS2411, chips:DS2411
- added X2: EPSON-FA-128, crystals:EPSON-FA-128
- added X3: FC-12M32.7680KA-A3, crystals:FC-12M32.7680KA-A3
Connections:
- removed net GPIOUNDECIDED: JP1.10
- removed net N$12: JP1.9
- new net !FRAM_CS: R3.1, U4.!CS, U5.PC5
- new net !FRAM_HOLD: R16.1, U4.!HOLD, U5.PC1
- new net !FRAM_WP: R19.1, U4.!WP, U5.PC6
- new net ANTENNA: A1.ANTENNA, B1.ANT
- new net DS2411: R22.1, U5.PC0, U6.I/O
- new net LED??: U5.PB4
- new net N$1: C29.1, C30.1, U5.DCOUPL1, U5.DCOUPL2
- new net N$10: C16.1, U5.XOSC32M_Q2, X2.2
- new net N$2: C32.1, R20.2, U5.!RESET
- new net N$6: C34.1, U5.PD7/XOSC32K_Q2, X3.2
- new net N$7: C33.1, U5.PD6/XOSC32K_Q1, X3.1
- new net N$8: R21.1, U5.R_BIAS
- new net N$9: C12.1, U5.XOSC32M_Q1, X2.1
- new net RF_N: B1.BAL_N, U5.RF_N
- new net RF_P: B1.BAL_P, U5.RF_P
- new net SCK: U4.SCK, U5.PC2
- new net TCK: J3.TCK, U5.JTAG_TCK
- new net TDI: U5.PB6/JTAG-TDI
- new net TDO: J3.TDO, U5.PB7/JTAG-TDO
- new net TMS: J3.TMS, U5.JTAG_TMS
- new net V_TIMER: U5.PA0/ROM-UART-RX
- net !ADE_CS: now also U5.PB2; no longer JP1.4
- net !ADE_IRQ: now also U5.PB1; no longer JP1.5
- net !RESET: now also J3.!RESET, R20.1
- net 3V3: now also C18.1, C19.1, C20.1, C21.1, C24.1, C25.1, C26.1, C27.1, C28.1, C31.1, J3.VCC, R16.2, R19.2, R22.2, R3.2, U4.VDD, U5.AVDD, U5.AVDD_GUARD, U5.DVDD, U6.VCC; no longer JP1.11
- net ADE_CF: now also U5.PC7; no longer JP1.7
- net ADE_ZX: now also U5.PB0; no longer JP1.6
- net GND: now also B1.GND, C12.2, C16.2, C18.2, C19.2, C20.2, C21.2, C24.2, C25.2, C26.2, C27.2, C28.2, C29.2, C30.2, C31.2, C32.2, C33.2, C34.2, J3.GND, R21.2, U4.VSS, U5.GND, U6.GND, X2.GND; no longer JP1.12
- net MISO: now also U4.SO, U5.PC4; no longer JP1.2
- net MOSI: now also U4.SI, U5.PC3; no longer JP1.1
- net RELAY_CTRL: now also U5.PB5
- net SCLK: no longer JP1.3
- net USER_RELAY_CTRL: now also U5.PB3; no longer JP1.8
Other:
- note added: "PIN10"
- note added: "PIN15"
- note added: "PIN24"
- note added: "PIN33"
- note added: "PIN36"
- note added: "PIN40"
- note added: "PIN43"
- note added: "PIN55"
- moved on the sheet: R7, S1

Commit message: working on ground plane
man there are some rediculous traces for this cc2538
Parts:
- added D4, D7: GREEN, SparkFun-LED:LED0603
- added D6: RED, SparkFun-LED:LED0603
- added R23, R24, R25: 470, passives:RESISTOR
- added U7: TXB0104RGY, chips:TXB0104RGY
Connections:
- removed net LED??: U5.PB4
- removed net SCK: U4.SCK, U5.PC2
- removed net V_TIMER: U5.PA0/ROM-UART-RX
- new net !ADE_CS_5V: U1.!CS, U7.B1
- new net GREEN_LED: D7.C, U5.PA6
- new net MISO_5V: U1.DOUT, U7.B3
- new net MOSI_5V: U1.DIN, U7.B4
- new net N$12: D4.A, R25.2
- new net N$20: D6.A, R23.2
- new net N$22: D7.A, R24.2
- new net RED_LED: D6.C, U5.PA7
- new net RELAY_LED: D4.C, U5.PB4
- new net SCLK_5V: U1.SCLK, U7.B2
- net !ADE_CS: now also U7.A1; no longer U1.!CS
- net 3V3: now also R23.1, R24.1, R25.1, U7.OE, U7.VCCA
- net 5V0: now also U7.VCCB
- net GND: now also U7.GND
- net MISO: now also U7.A3; no longer U1.DOUT
- net MOSI: now also U7.A4; no longer U1.DIN
- net SCLK: now also U4.SCK, U5.PC2, U7.A2; no longer U1.SCLK
Other:
- moved on the sheet: R7, S1

Commit message: routed.
still not sure what to do with "GND" for the differential signals
running to the ade
Connections:
- new net !ADE_RESET: R8.2, U1.!RESET
- new net N$19: C22.2
- new net N$23: C13.2
- new net N$25: C23.2
- new net N$27: R15.1
- net !RESET: no longer R8.2, U1.!RESET
- net GND: no longer C13.2, C22.2, C23.2, R15.1
Changed lines of the file:
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@@
 <attribute name="DIGIKEY" value="478-1389-1-ND"/>
 </part>
-<part name="GND7" library="supply1" deviceset="GND" device=""/>
-<part name="GND12" library="supply1" deviceset="GND" device=""/>
 <part name="L4" library="powercube" deviceset="35F0121-0SR-10" device=""/>
 <part name="R14" library="SparkFun-Resistors" deviceset="RESISTOR" device="0805-RES" value="499k">
@@
 <attribute name="DIGIKEY" value="RHM1.00KADCT-ND"/>
 </part>
-<part name="GND17" library="supply1" deviceset="GND" device=""/>
 <part name="C23" library="SparkFun-Passives" deviceset="CAP" device="0805" value="33nF">
 <attribute name="DIGIKEY" value="478-1389-1-ND"/>
 </part>
-<part name="GND18" library="supply1" deviceset="GND" device=""/>
 <part name="J1" library="powercube" deviceset="AC-PLUG" device=""/>
 <part name="J2" library="powercube" deviceset="WIRE_HOLE-14AWG" device=""/>
@@
 </segment>
 </net>
-<net name="!RESET" class="0">
-<segment>
-<pinref part="U1" gate="G$1" pin="!RESET"/>
-<wire x1="114.3" y1="132.08" x2="111.76" y2="132.08" width="0.1524" layer="91"/>
-<wire x1="111.76" y1="132.08" x2="109.22" y2="132.08" width="0.1524" layer="91"/>
-<wire x1="111.76" y1="132.08" x2="111.76" y2="137.16" width="0.1524" layer="91"/>
-<junction x="111.76" y="132.08"/>
-<pinref part="R8" gate="G$1" pin="2"/>
-<label x="109.22" y="132.08" size="1.27" layer="95" rot="R180" xref="yes"/>
-</segment>
-</net>
 <net name="V1P" class="0">
 <segment>
@@
 </segment>
 </net>
+<net name="!ADE_RESET" class="0">
+<segment>
+<pinref part="U1" gate="G$1" pin="!RESET"/>
+<wire x1="114.3" y1="132.08" x2="111.76" y2="132.08" width="0.1524" layer="91"/>
+<wire x1="111.76" y1="132.08" x2="109.22" y2="132.08" width="0.1524" layer="91"/>
+<wire x1="111.76" y1="132.08" x2="111.76" y2="137.16" width="0.1524" layer="91"/>
+<junction x="111.76" y="132.08"/>
+<pinref part="R8" gate="G$1" pin="2"/>
+<label x="109.22" y="132.08" size="1.27" layer="95" rot="R180" xref="yes"/>
+</segment>
+</net>
 </nets>
 </sheet>
@@
 <attribute name="DIGIKEY" x="91.44" y="147.32" size="1.27" layer="96" display="off"/>
 </instance>
-<instance part="GND7" gate="1" x="91.44" y="111.76"/>
-<instance part="GND12" gate="1" x="91.44" y="139.7"/>
 <instance part="L4" gate="G$1" x="45.72" y="91.44"/>
 <instance part="R14" gate="G$1" x="68.58" y="91.44">
@@
 <attribute name="DIGIKEY" x="78.74" y="81.28" size="1.27" layer="96" rot="R90" display="off"/>
 </instance>
-<instance part="GND17" gate="1" x="78.74" y="68.58"/>
 <instance part="C23" gate="G$1" x="88.9" y="81.28">
 <attribute name="DIGIKEY" x="88.9" y="81.28" size="1.27" layer="96" display="off"/>
 </instance>
-<instance part="GND18" gate="1" x="88.9" y="68.58"/>
 <instance part="J1" gate="G$1" x="147.32" y="167.64"/>
 <instance part="J2" gate="G$1" x="223.52" y="170.18" smashed="yes" rot="R180">
@@
 <wire x1="40.64" y1="15.24" x2="40.64" y2="12.7" width="0.1524" layer="91"/>
 <pinref part="GND6" gate="1" pin="GND"/>
-</segment>
-<segment>
-<pinref part="C13" gate="G$1" pin="2"/>
-<wire x1="91.44" y1="116.84" x2="91.44" y2="114.3" width="0.1524" layer="91"/>
-<pinref part="GND7" gate="1" pin="GND"/>
-</segment>
-<segment>
-<pinref part="C22" gate="G$1" pin="2"/>
-<wire x1="91.44" y1="144.78" x2="91.44" y2="142.24" width="0.1524" layer="91"/>
-<pinref part="GND12" gate="1" pin="GND"/>
-</segment>
-<segment>
-<pinref part="R15" gate="G$1" pin="1"/>
-<wire x1="78.74" y1="76.2" x2="78.74" y2="71.12" width="0.1524" layer="91"/>
-<pinref part="GND17" gate="1" pin="GND"/>
-</segment>
-<segment>
-<pinref part="C23" gate="G$1" pin="2"/>
-<wire x1="88.9" y1="78.74" x2="88.9" y2="71.12" width="0.1524" layer="91"/>
-<pinref part="GND18" gate="1" pin="GND"/>
 </segment>
 </net>
@@
 <wire x1="40.64" y1="48.26" x2="40.64" y2="50.8" width="0.1524" layer="91"/>
 <pinref part="5V3" gate="1" pin="5V0"/>
+</segment>
+</net>
+<net name="N$19" class="0">
+<segment>
+<pinref part="C22" gate="G$1" pin="2"/>
+<wire x1="91.44" y1="144.78" x2="91.44" y2="142.24" width="0.1524" layer="91"/>
+</segment>
+</net>
+<net name="N$23" class="0">
+<segment>
+<pinref part="C13" gate="G$1" pin="2"/>
+<wire x1="91.44" y1="116.84" x2="91.44" y2="114.3" width="0.1524" layer="91"/>
+</segment>
+</net>
+<net name="N$25" class="0">
+<segment>
+<pinref part="C23" gate="G$1" pin="2"/>
+<wire x1="88.9" y1="78.74" x2="88.9" y2="71.12" width="0.1524" layer="91"/>
+</segment>
+</net>
+<net name="N$27" class="0">
+<segment>
+<pinref part="R15" gate="G$1" pin="1"/>
+<wire x1="78.74" y1="76.2" x2="78.74" y2="71.12" width="0.1524" layer="91"/>
 </segment>
 </net>
@@
 <instance part="U2" gate="G$1" x="109.22" y="111.76"/>
 <instance part="D3" gate="G$1" x="53.34" y="160.02"/>
-<instance part="GND2" gate="1" x="60.96" y="147.32"/>
+<instance part="GND2" gate="1" x="60.96" y="91.44"/>
 <instance part="R1" gate="G$1" x="81.28" y="154.94" rot="R90">
 <attribute name="DIGIKEY" x="81.28" y="154.94" size="1.27" layer="96" rot="R90" display="off"/>
@@
 <attribute name="DIGIKEY" x="81.28" y="142.24" size="1.27" layer="96" rot="R90" display="off"/>
 </instance>
-<instance part="GND8" gate="1" x="81.28" y="132.08"/>
+<instance part="GND8" gate="1" x="81.28" y="91.44"/>
 <instance part="R4" gate="G$1" x="91.44" y="154.94" rot="R90">
 <attribute name="DIGIKEY" x="91.44" y="154.94" size="1.27" layer="96" rot="R90" display="off"/>
@@
 <pinref part="D3" gate="G$1" pin="NEG"/>
 <wire x1="58.42" y1="157.48" x2="60.96" y2="157.48" width="0.1524" layer="91"/>
-<wire x1="60.96" y1="157.48" x2="60.96" y2="149.86" width="0.1524" layer="91"/>
+<wire x1="60.96" y1="157.48" x2="60.96" y2="93.98" width="0.1524" layer="91"/>
 <pinref part="GND2" gate="1" pin="GND"/>
 </segment>
 <segment>
 <pinref part="R2" gate="G$1" pin="1"/>
-<wire x1="81.28" y1="137.16" x2="81.28" y2="134.62" width="0.1524" layer="91"/>
+<wire x1="81.28" y1="137.16" x2="81.28" y2="93.98" width="0.1524" layer="91"/>
 <pinref part="GND8" gate="1" pin="GND"/>
 </segment>
