File: hardware/ACme++/rev_b/ACme++.brd (EAGLE design)
At the start: 72.6 x 47.1 mm, 98 parts, among them J1 HOLE, J3 WIRE_HOLE-14AWG, J4 WIRE_HOLE-14AWG, J6 HOLE, J7 HOLE, J8 HOLE, J9 TC2030-CC2538-BL-NL, K1 S216S01F, Q1 STGD5NB120SZT4, Q2 FDV301N, U1 CC2538, U3 FM25LBTDFN-8, U4 ADE7753, U5 TXB0104RGY, U6 SR086SG-G, U7 TDA3664AT, X1 EPSON-FA-128, X2 FC-12M32.7680KA-A3, X3 ECS-35-17-5PX-TR

Commit message: acme ++ rev b changes
Parts:
- added TP10, TP11, TP8, TP9: TEST_POINT_0.040IN, headers:TESTPOINT_0.040IN
- added TP12, TP13, TP14: TPTP09SQ, testpad:TP09SQ
- moved C6 2.29 mm to (17.6, 41.5), turned to 270 degrees
- moved U5 0.18 mm to (19.1, 34.5)
- moved X3 0.13 mm to (24.1, 44.5)
Connections:
- new net TCK: TP14.TP, U1.47
- new net TDO: TP13.TP, U1.48
- new net TMS: TP12.TP, U1.46
- net !ADE_IRQ: now also TP9.TESTPOINT
- net ADE_CF: now also TP11.TESTPOINT
- net ADE_ZX: now also TP10.TESTPOINT
- net GND: now also TP8.TESTPOINT
Routing:
- net TDO: track 0.00 -> 5.22 mm
- net TMS: track 0.00 -> 3.60 mm
- net N$3: track 11.9 -> 14.0 mm
- net 3V3: track 163.7 -> 161.9 mm
- net TCK: track 0.00 -> 1.56 mm
- net ADE_ZX: track 18.9 -> 20.2 mm
- net ADE_CF: track 19.7 -> 20.9 mm
- net !ADE_IRQ: track 20.6 -> 21.6 mm
- net 5V0: track 46.7 -> 46.0 mm
- net GND: vias 104 -> 101
Other:
- board text added: "!IRQ"
- board text added: "CF"
- board text added: "GND"
- board text added: "TCK"
- board text added: "TDO"
- board text added: "TMS"
- board text added: "ZX"

Commit message: new version of acme++
Parts:
- removed R25: 510k, SparkFun-Resistors:1206
- removed U7: TDA3664AT, powercube:SOIC_8
- added L4: MPZ2012S300A, powercube:0805_RESISTOR
- added R10: 2.2k, passives:0402_RES
- added U2: FM25LBTDFN-8, chips:TDFN-8
- R11: value 2.2k -> 4.7k
- R14: value 4.7k -> 10k; device passives:0402_RES -> SparkFun:0603-RES
- R16: value 10k -> 12.4k; device SparkFun:0603-RES -> SparkFun-Resistors:0603-RES
- R17: value 12.4k -> 56k; device SparkFun-Resistors:0603-RES -> passives:0402_RES
- R18: value 56k -> 100k; device passives:0402_RES -> SparkFun:0603-RES
- R19: value 100k -> 113k; device SparkFun:0603-RES -> SparkFun-Resistors:0603-RES
- R20: value 113k -> 200k; device SparkFun-Resistors:0603-RES -> SparkFun-Resistors:1206
- R22: value 200k -> 499k; device SparkFun-Resistors:1206 -> SparkFun-Resistors:0805
- R23: value 499k -> 510k; device SparkFun-Resistors:0805 -> SparkFun-Resistors:1206
- U3: value FM25LBTDFN-8 -> ADE7753; device chips:TDFN-8 -> powercube:SSOP-20
- U4: value ADE7753 -> TXB0104RGY; device powercube:SSOP-20 -> chips:S-PVQFN-N14
- U5: value TXB0104RGY -> SR086SG-G; device chips:S-PVQFN-N14 -> powercube:SR086
- U6: value SR086SG-G -> TDA3664AT; device powercube:SR086 -> powercube:SOIC_8
- moved U5 32.8 mm to (37.2, 7.24)
- moved R16 28.8 mm to (36.3, 3.81), turned to 0 degrees
- moved R22 26.9 mm to (49.1, 32.4), turned to 90 degrees
- moved R17 26.9 mm to (14.4, 19.3), turned to 270 degrees
- moved R14 23.4 mm to (26.7, 18.9), turned to 0 degrees
- moved R23 21.9 mm to (41.8, 11.8), turned to 0 degrees
- moved R20 20.8 mm to (58.3, 11.4), turned to 90 degrees
- moved TP8 18.6 mm to (20.5, 40.6)
- moved U3 18.0 mm to (26.0, 37.0), turned to 180 degrees
- moved TP11 17.7 mm to (37.8, 36.7)
- moved TP7 17.4 mm to (20.5, 37.9)
- moved TP6 17.3 mm to (17.8, 37.9)
- moved R18 17.2 mm to (31.2, 16.0)
- moved TP5 17.1 mm to (15.4, 39.4)
- moved R19 15.6 mm to (39.4, 2.67), turned to 0 degrees
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Connections:
- net !ADE_CS: now also TP5.TESTPOINT, U4.2; no longer TP4.TESTPOINT, U5.2
- net !ADE_CS_5V: now also U3.17, U4.13; no longer U4.17, U5.13
- net !ADE_IRQ: now also TP6.TESTPOINT, U3.14; no longer TP9.TESTPOINT, U4.14
- net !ADE_RESET: now also R15.2, U3.1; no longer R16.2, U4.1
- net !FRAM_CS: now also R11.1, U2.1; no longer R12.1, U3.1
- net !FRAM_HOLD: now also R12.1, U2.7; no longer R13.1, U3.7
- net !FRAM_WP: now also R13.1, U2.3; no longer R14.1, U3.3
- net !RESET: now also R10.1; no longer R11.1
- net 3V3: now also R11.2, R18.1, U2.8, U4.1, U4.8, U5.4; no longer R14.2, R19.1, U3.8, U5.1, U5.8, U6.4
- net 5V0: now also R15.1, U3.2, U4.14, U6.1; no longer R16.1, U4.2, U5.14, U7.1
- net ADE_AVDD: now also U3.3; no longer U4.3
- net ADE_CF: now also TP8.TESTPOINT, U3.11; no longer TP11.TESTPOINT, U4.11
- net ADE_ZX: now also TP7.TESTPOINT, U3.12; no longer TP10.TESTPOINT, U4.12
- net DC_RECTIFIED: now also R20.2, R23.2; no longer R21.2, R24.2
- net GND: now also L4.P$2, R14.1, R16.1, R17.2, R21.1, TP1.TESTPOINT, U2.4, U3.10, U3.8, U4.7, U4.THERMALPAD, U5.2, U5.3, U5.PAD; no longer R15.1, R17.1, R18.2, R22.1, TP8.TESTPOINT, U3.4, U4.10, U4.8, U5.7, U5.THERMALPAD, U6.2, U6.PAD, U7.3
- net MISO: now also TP3.TESTPOINT, U2.2, U4.4; no longer TP2.TESTPOINT, U3.2, U5.4
- net MISO_5V: now also U3.19, U4.11; no longer U4.19, U5.11
- net MOSI: now also TP2.TESTPOINT, U2.5, U4.5; no longer TP1.TESTPOINT, U3.5, U5.5
- net MOSI_5V: now also U3.20, U4.10; no longer U4.20, U5.10
- net N$11: now also U3.9; no longer U4.9
- net N$15: now also U3.16; no longer U4.16
- net N$17: now also R22.1; no longer R23.1
- net N$18: now also R20.1, R21.2; no longer R21.1, R22.2
- net N$2: now also R10.2; no longer R11.2
- net N$21: now also R23.1, R24.2; no longer R24.1, R25.2
- net N$24: now also U5.7; no longer U6.7
- net N$26: now also R16.2, R19.1, U5.5; no longer R17.2, R20.1, U6.5
- net N$3: now also U3.15; no longer U4.15
- net N$8: now also R17.1; no longer R18.1
- net RELAY_CTRL: now also R18.2; no longer R19.2
- net SCLK: now also TP4.TESTPOINT, U2.6, U4.3; no longer TP3.TESTPOINT, U3.6, U5.3
- net SCLK_5V: now also U3.18, U4.12; no longer U4.18, U5.12
- net SR086_GATE: now also U5.8; no longer U6.8
- net SR086_VIN: now also R24.1, U5.1; no longer R25.1, U6.1
- net USER_RELAY_CTRL: now also R14.2; no longer R15.2
- net V1N: now also TP10.TESTPOINT, U3.5, U3.6; no longer TP6.TESTPOINT, U4.5, U4.6
- net V1P: now also TP9.TESTPOINT, U3.4; no longer TP5.TESTPOINT, U4.4
- net V2P: now also R22.2, TP11.TESTPOINT, U3.7; no longer R23.2, TP7.TESTPOINT, U4.7
- net VDC: now also R19.2, U5.6, U6.8; no longer R20.2, U6.6, U7.8
- net WALL_NEUTRAL: now also L4.P$1
Routing:
- net GND: track 57.6 -> 76.7 mm
- net WALL_NEUTRAL: track 19.4 -> 25.7 mm
- net RF_P: track 0.00 -> 3.99 mm
- net RF_N: track 0.00 -> 3.98 mm
- net WALL_PHASE: track 56.0 -> 53.1 mm
- net ANTENNA: track 0.00 -> 2.51 mm
- net N$18: track 3.17 -> 2.41 mm
- removed copper zone on layer 1, net ANTENNA
- removed copper zone on layer 1, net RF_N
- removed copper zone on layer 1, net RF_P
Other:
- board text added: "2014/08/20"
- board text removed: "2014/08/13"
