File: hardware/ACme++/rev_b/ACme++.sch (EAGLE design)
At the start: 98 parts, among them J1 HOLE, J3 WIRE_HOLE-14AWG, J4 WIRE_HOLE-14AWG, J6 HOLE, J7 HOLE, J8 HOLE, J9 TC2030-CC2538-BL-NL, K1 S216S01F, Q1 STGD5NB120SZT4, Q2 FDV301N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

Commit message: acme ++ rev b changes
Parts:
- added TP10, TP11, TP8, TP9: TEST_POINT_0.040IN, headers:TEST_POINT_0.040IN
- added TP12, TP13, TP14: TPTP09SQ, testpad:TPTP09SQ
Connections:
- new net TCK: TP14.TP, U1.JTAG_TCK
- new net TDO: TP13.TP, U1.PB7/JTAG-TDO
- new net TMS: TP12.TP, U1.JTAG_TMS
- net !ADE_IRQ: now also TP9.TESTPOINT
- net ADE_CF: now also TP11.TESTPOINT
- net ADE_ZX: now also TP10.TESTPOINT
- net GND: now also TP8.TESTPOINT
Changed lines of the file:
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@@
 <part name="3V5" library="powercube" deviceset="3V3" device=""/>
 <part name="GND2" library="supply1" deviceset="GND" device=""/>
+<part name="TP8" library="headers" deviceset="TEST_POINT_0.040IN" device=""/>
+<part name="TP9" library="headers" deviceset="TEST_POINT_0.040IN" device=""/>
+<part name="TP10" library="headers" deviceset="TEST_POINT_0.040IN" device=""/>
+<part name="TP11" library="headers" deviceset="TEST_POINT_0.040IN" device=""/>
+<part name="TP14" library="testpad" deviceset="TP" device="TP09SQ"/>
+<part name="TP12" library="testpad" deviceset="TP" device="TP09SQ"/>
+<part name="TP13" library="testpad" deviceset="TP" device="TP09SQ"/>
 </parts>
 <sheets>
@@
 <instance part="3V5" gate="G$1" x="45.72" y="167.64"/>
 <instance part="GND2" gate="1" x="45.72" y="152.4"/>
+<instance part="TP8" gate="G$1" x="63.5" y="17.78" rot="R180"/>
+<instance part="TP14" gate="G$1" x="86.36" y="55.88" smashed="yes">
+<attribute name="NAME" x="87.122" y="55.88" size="1.778" layer="95" rot="R90"/>
+<attribute name="TP_SIGNAL_NAME" x="87.63" y="54.61" size="1.778" layer="97"/>
+</instance>
+<instance part="TP12" gate="G$1" x="88.9" y="55.88" smashed="yes">
+<attribute name="NAME" x="89.662" y="55.88" size="1.778" layer="95" rot="R90"/>
+<attribute name="TP_SIGNAL_NAME" x="90.17" y="54.61" size="1.778" layer="97"/>
+</instance>
+<instance part="TP13" gate="G$1" x="10.16" y="63.5" smashed="yes">
+<attribute name="NAME" x="9.144" y="60.96" size="1.778" layer="95" rot="R90"/>
+<attribute name="TP_SIGNAL_NAME" x="11.43" y="62.23" size="1.778" layer="97"/>
+</instance>
 </instances>
 <busses>
@@
 <segment>
 <pinref part="U1" gate="G$1" pin="GND"/>
-<wire x1="58.42" y1="25.4" x2="58.42" y2="15.24" width="0.1524" layer="91"/>
+<wire x1="58.42" y1="25.4" x2="58.42" y2="17.78" width="0.1524" layer="91"/>
 <pinref part="GND27" gate="1" pin="GND"/>
+<pinref part="TP8" gate="G$1" pin="TESTPOINT"/>
+<wire x1="58.42" y1="17.78" x2="58.42" y2="15.24" width="0.1524" layer="91"/>
+<wire x1="60.96" y1="17.78" x2="58.42" y2="17.78" width="0.1524" layer="91"/>
+<junction x="58.42" y="17.78"/>
 </segment>
 <segment>
@@
 </segment>
 </net>
+<net name="TCK" class="0">
+<segment>
+<pinref part="U1" gate="G$1" pin="JTAG_TCK"/>
+<wire x1="83.82" y1="50.8" x2="86.36" y2="50.8" width="0.1524" layer="91"/>
+<label x="91.44" y="50.8" size="1.27" layer="95" xref="yes"/>
+<pinref part="TP14" gate="G$1" pin="TP"/>
+<wire x1="86.36" y1="50.8" x2="91.44" y2="50.8" width="0.1524" layer="91"/>
+<wire x1="86.36" y1="53.34" x2="86.36" y2="50.8" width="0.1524" layer="91"/>
+<junction x="86.36" y="50.8"/>
+</segment>
+<segment>
+<wire x1="132.08" y1="154.94" x2="137.16" y2="154.94" width="0.1524" layer="91"/>
+<label x="137.16" y="154.94" size="1.27" layer="95" xref="yes"/>
+</segment>
+</net>
+<net name="TMS" class="0">
+<segment>
+<pinref part="U1" gate="G$1" pin="JTAG_TMS"/>
+<wire x1="83.82" y1="48.26" x2="88.9" y2="48.26" width="0.1524" layer="91"/>
+<label x="91.44" y="48.26" size="1.27" layer="95" xref="yes"/>
+<pinref part="TP12" gate="G$1" pin="TP"/>
+<wire x1="88.9" y1="48.26" x2="91.44" y2="48.26" width="0.1524" layer="91"/>
+<wire x1="88.9" y1="53.34" x2="88.9" y2="48.26" width="0.1524" layer="91"/>
+<junction x="88.9" y="48.26"/>
+</segment>
+<segment>
+<wire x1="132.08" y1="152.4" x2="137.16" y2="152.4" width="0.1524" layer="91"/>
+<label x="137.16" y="152.4" size="1.27" layer="95" xref="yes"/>
+</segment>
+</net>
+<net name="TDO" class="0">
+<segment>
+<pinref part="U1" gate="G$1" pin="PB7/JTAG-TDO"/>
+<wire x1="33.02" y1="58.42" x2="10.16" y2="58.42" width="0.1524" layer="91"/>
+<label x="7.62" y="58.42" size="1.27" layer="95" rot="R180" xref="yes"/>
+<pinref part="TP13" gate="G$1" pin="TP"/>
+<wire x1="10.16" y1="58.42" x2="7.62" y2="58.42" width="0.1524" layer="91"/>
+<wire x1="10.16" y1="60.96" x2="10.16" y2="58.42" width="0.1524" layer="91"/>
+<junction x="10.16" y="58.42"/>
+</segment>
+<segment>
+<wire x1="132.08" y1="157.48" x2="137.16" y2="157.48" width="0.1524" layer="91"/>
+<label x="137.16" y="157.48" size="1.27" layer="95" xref="yes"/>
+</segment>
+</net>
 </nets>
 </sheet>
@@
 <instance part="TP3" gate="G$1" x="43.18" y="58.42" rot="R270"/>
 <instance part="TP4" gate="G$1" x="45.72" y="58.42" rot="R270"/>
+<instance part="TP9" gate="G$1" x="152.4" y="104.14" rot="R90"/>
+<instance part="TP10" gate="G$1" x="154.94" y="104.14" rot="R90"/>
+<instance part="TP11" gate="G$1" x="157.48" y="104.14" rot="R90"/>
 </instances>
 <busses>
@@
 <segment>
 <pinref part="U4" gate="G$1" pin="!IRQ"/>
+<wire x1="154.94" y1="116.84" x2="152.4" y2="116.84" width="0.1524" layer="91"/>
+<label x="154.94" y="116.84" size="1.27" layer="95" xref="yes"/>
+<pinref part="TP9" gate="G$1" pin="TESTPOINT"/>
 <wire x1="152.4" y1="116.84" x2="149.86" y2="116.84" width="0.1524" layer="91"/>
-<label x="152.4" y="116.84" size="1.27" layer="95" xref="yes"/>
+<wire x1="152.4" y1="106.68" x2="152.4" y2="116.84" width="0.1524" layer="91"/>
+<junction x="152.4" y="116.84"/>
 </segment>
 </net>
@@
 <segment>
 <pinref part="U4" gate="G$1" pin="ZX"/>
-<wire x1="152.4" y1="111.76" x2="149.86" y2="111.76" width="0.1524" layer="91"/>
-<label x="152.4" y="111.76" size="1.27" layer="95" xref="yes"/>
+<wire x1="160.02" y1="111.76" x2="154.94" y2="111.76" width="0.1524" layer="91"/>
+<label x="160.02" y="111.76" size="1.27" layer="95" xref="yes"/>
+<pinref part="TP10" gate="G$1" pin="TESTPOINT"/>
+<wire x1="154.94" y1="111.76" x2="149.86" y2="111.76" width="0.1524" layer="91"/>
+<wire x1="154.94" y1="106.68" x2="154.94" y2="111.76" width="0.1524" layer="91"/>
+<junction x="154.94" y="111.76"/>
 </segment>
 </net>
@@
 <segment>
 <pinref part="U4" gate="G$1" pin="CF"/>
-<wire x1="152.4" y1="109.22" x2="149.86" y2="109.22" width="0.1524" layer="91"/>
-<label x="152.4" y="109.22" size="1.27" layer="95" xref="yes"/>
-</segment>
-</net>
+<wire x1="160.02" y1="109.22" x2="157.48" y2="109.22" width="0.1524" layer="91"/>
+<label x="160.02" y="109.22" size="1.27" layer="95" xref="yes"/>
+<pinref part="TP11" gate="G$1" pin="TESTPOINT"/>
+<wire x1="157.48" y1="109.22" x2="149.86" y2="109.22" width="0.1524" layer="91"/>
+<wire x1="157.48" y1="106.68" x2="157.48" y2="109.22" width="0.1524" layer="91"/>
+<junction x="157.48" y="109.22"/>
+</segment>
+</net>

Commit message: new version of acme++
Parts:
- removed R25: 510k, SparkFun-Resistors:RESISTOR1206
- removed U7: TDA3664AT, powercube:TDA3664AT
- added L4: MPZ2012S300A, powercube:MPZ2012S300A
- added R10: 2.2k, passives:RESISTOR
- added U2: FM25LBTDFN-8, chips:FM25LBTDFN-8
- R11: value 2.2k -> 4.7k; DIGIKEY RHM2.2KCECT-ND -> RHM4.7KCECT-ND
- R14: value 4.7k -> 10k; device passives:RESISTOR -> SparkFun:RESISTOR0603-RES; DIGIKEY RHM4.7KCECT-ND -> RHM10.0KCFCT-ND
- R16: value 10k -> 12.4k; device SparkFun:RESISTOR0603-RES -> SparkFun-Resistors:RESISTOR0603-RES; DIGIKEY RHM10.0KCFCT-ND -> RHM12.4KCFCT-ND
- R17: value 12.4k -> 56k; device SparkFun-Resistors:RESISTOR0603-RES -> passives:RESISTOR; DIGIKEY RHM12.4KCFCT-ND -> RHM56KBHCT-ND
- R18: value 56k -> 100k; device passives:RESISTOR -> SparkFun:RESISTOR0603-RES; DIGIKEY RHM56KBHCT-ND -> RHM100KCGCT-ND
- R19: value 100k -> 113k; device SparkFun:RESISTOR0603-RES -> SparkFun-Resistors:RESISTOR0603-RES; DIGIKEY RHM100KCGCT-ND -> RHM113KCFCT-ND
- R20: value 113k -> 200k; device SparkFun-Resistors:RESISTOR0603-RES -> SparkFun-Resistors:RESISTOR1206; DIGIKEY RHM113KCFCT-ND -> P200KALCT-ND
- R22: value 200k -> 499k; device SparkFun-Resistors:RESISTOR1206 -> SparkFun-Resistors:RESISTOR0805-RES; DIGIKEY P200KALCT-ND -> P499KCCT-ND
- R23: value 499k -> 510k; device SparkFun-Resistors:RESISTOR0805-RES -> SparkFun-Resistors:RESISTOR1206; DIGIKEY P499KCCT-ND -> P510KALCT-ND
- U3: value FM25LBTDFN-8 -> ADE7753; device chips:FM25LBTDFN-8 -> powercube:ADE7753; DIGIKEY FM25L04B-DGRA-ND -> (none); MOUSER 877-FM25L04B-DG -> 584-ADE7753ARSZR
- U4: value ADE7753 -> TXB0104RGY; device powercube:ADE7753 -> chips:TXB0104RGY; MOUSER 584-ADE7753ARSZR -> (none)
- U5: value TXB0104RGY -> SR086SG-G; device chips:TXB0104RGY -> powercube:SR086SG-G
- U6: value SR086SG-G -> TDA3664AT; device powercube:SR086SG-G -> powercube:TDA3664AT
Connections:
- net !ADE_CS: now also TP5.TESTPOINT, U4.A1; no longer TP4.TESTPOINT, U5.A1
- net !ADE_CS_5V: now also U3.!CS, U4.B1; no longer U4.!CS, U5.B1
- net !ADE_IRQ: now also TP6.TESTPOINT, U3.!IRQ; no longer TP9.TESTPOINT, U4.!IRQ
- net !ADE_RESET: now also R15.2, U3.!RESET; no longer R16.2, U4.!RESET
- net !FRAM_CS: now also R11.1, U2.!CS; no longer R12.1, U3.!CS
- net !FRAM_HOLD: now also R12.1, U2.!HOLD; no longer R13.1, U3.!HOLD
- net !FRAM_WP: now also R13.1, U2.!WP; no longer R14.1, U3.!WP
- net !RESET: now also R10.1; no longer R11.1
- net 3V3: now also R11.2, R18.1, U2.VDD, U4.OE, U4.VCCA, U5.VREG; no longer R14.2, R19.1, U3.VDD, U5.OE, U5.VCCA, U6.VREG
- net 5V0: now also R15.1, U3.DVDD, U4.VCCB, U6.VOUT; no longer R16.1, U4.DVDD, U5.VCCB, U7.VOUT
- net ADE_AVDD: now also U3.AVDD; no longer U4.AVDD
- net ADE_CF: now also TP8.TESTPOINT, U3.CF; no longer TP11.TESTPOINT, U4.CF
- net ADE_ZX: now also TP7.TESTPOINT, U3.ZX; no longer TP10.TESTPOINT, U4.ZX
- net DC_RECTIFIED: now also R20.2, R23.2; no longer R21.2, R24.2
- net GND: now also L4.P$2, R14.1, R16.1, R17.2, R21.1, TP1.TESTPOINT, U2.VSS, U3.AGND, U3.DGND, U4.GND, U5.!EN; no longer R15.1, R17.1, R18.2, R22.1, TP8.TESTPOINT, U3.VSS, U4.AGND, U4.DGND, U6.!EN, U7.GND
- net MISO: now also TP3.TESTPOINT, U2.SO, U4.A3; no longer TP2.TESTPOINT, U3.SO, U5.A3
- net MISO_5V: now also U3.DOUT, U4.B3; no longer U4.DOUT, U5.B3
- net MOSI: now also TP2.TESTPOINT, U2.SI, U4.A4; no longer TP1.TESTPOINT, U3.SI, U5.A4
- net MOSI_5V: now also U3.DIN, U4.B4; no longer U4.DIN, U5.B4
- net N$11: now also U3.REF; no longer U4.REF
- net N$15: now also U3.CLKOUT; no longer U4.CLKOUT
- net N$17: now also R22.1; no longer R23.1
- net N$18: now also R20.1, R21.2; no longer R21.1, R22.2
- net N$2: now also R10.2; no longer R11.2
- net N$21: now also R23.1, R24.2; no longer R24.1, R25.2
- net N$24: now also U5.VGD; no longer U6.VGD
- net N$26: now also R16.2, R19.1, U5.FB; no longer R17.2, R20.1, U6.FB
- net N$3: now also U3.CLKIN; no longer U4.CLKIN
- net N$8: now also R17.1; no longer R18.1
- net RELAY_CTRL: now also R18.2; no longer R19.2
- net SCLK: now also TP4.TESTPOINT, U2.SCK, U4.A2; no longer TP3.TESTPOINT, U3.SCK, U5.A2
- net SCLK_5V: now also U3.SCLK, U4.B2; no longer U4.SCLK, U5.B2
- net SR086_GATE: now also U5.GATE; no longer U6.GATE
- net SR086_VIN: now also R24.1, U5.VIN; no longer R25.1, U6.VIN
- net USER_RELAY_CTRL: now also R14.2; no longer R15.2
- net V1N: now also TP10.TESTPOINT, U3.V1N, U3.V2N; no longer TP6.TESTPOINT, U4.V1N, U4.V2N
- net V1P: now also TP9.TESTPOINT, U3.V1P; no longer TP5.TESTPOINT, U4.V1P
- net V2P: now also R22.2, TP11.TESTPOINT, U3.V2P; no longer R23.2, TP7.TESTPOINT, U4.V2P
- net VDC: now also R19.2, U5.VOUT, U6.VIN; no longer R20.2, U6.VOUT, U7.VIN
- net WALL_NEUTRAL: now also L4.P$1
Other:
- moved on the sheet: R11, R12, R13, R14, R20, R21, R24, TP2, TP3, TP4
